Commit message: updated two sensor urdf.xacro to new standard

File: urdf/hokuyo_ust10lx.urdf.xacro (robot description, xacro)
@@ -1,12 +1,11 @@
 <?xml version="1.0"?>
 <robot name="sensor_hokuyo_ust10lx" xmlns:xacro="http://www.ros.org/wiki/xacro">
-  <xacro:macro name="sensor_hokuyo_ust10lx" params="prefix_frame prefix_topic parent *origin min_angle:=-2.3562 max_angle:=2.3562">
-			<!--arg name="namespace" value="$(arg namespace)"/-->
-    <joint name="${prefix_frame}_joint" type="fixed">
+  <xacro:macro name="sensor_hokuyo_ust10lx" params="name parent *origin min_angle:=-2.3562 max_angle:=2.3562">
+    <joint name="${name}_joint" type="fixed">
       <xacro:insert_block name="origin" />
       <parent link="${parent}"/>
-      <child link="${prefix_frame}_link"/>
+      <child link="${name}_link"/>
     </joint>
-    <link name="${prefix_frame}_link">
+    <link name="${name}_link">
       <collision>
         <origin xyz="0 0 -0.05" rpy="0 0 0"/>
@@ -31,6 +30,6 @@
   </xacro:macro>
   <xacro:macro name="sensor_hokuyo_ust_gazebo">
-    <gazebo reference="${prefix_frame}_link">
-			<sensor type="ray" name="${prefix_frame}_sensor">
+    <gazebo reference="${name}_link">
+			<sensor type="ray" name="${name}_sensor">
 				<pose>0 0 0 0 0 0</pose>
 				<visualize>false</visualize>
@@ -58,8 +57,12 @@
 					</noise>
 				</ray>
-				<plugin name="${prefix_frame}_controller" filename="libgazebo_ros_laser.so">
+				<!-- plugin name="${name}_controller" filename="libgazebo_ros_laser.so">
 					<topicName>${prefix_topic}hokuyo_base/scan</topicName>
-					<frameName>${prefix_frame}_link</frameName>
+					<frameName>${name}_link</frameName>
 					<ignoreTfPrefix>1</ignoreTfPrefix>
+				</plugin -->
+				<plugin name="${name}_controller" filename="libgazebo_ros_laser.so">
+					<topicName>${name}/scan</topicName>
+					<frameName>${name}_link</frameName>
 				</plugin>
 			</sensor>

File: urdf/imu_hector_plugin.urdf.xacro (robot description, xacro)
@@ -1,13 +1,12 @@
 <?xml version="1.0"?>
 <robot name="sensor_imu" xmlns:xacro="http://www.ros.org/wiki/xacro">
-  <xacro:macro name="sensor_imu_hector" params="prefix_frame prefix_topic parent *origin">
-	  <joint name="${prefix_frame}_joint" type="fixed">
+  <xacro:macro name="sensor_imu_hector" params="name parent *origin">
+	  <joint name="${name}_joint" type="fixed">
 	      <axis xyz="1 0 0"/>
-	      <!--origin xyz="0 0 0.2825"/-->
 	      <xacro:insert_block name="origin"/>
 	      <parent link="${parent}"/>
-	      <child link="${prefix_frame}_link"/>
+	      <child link="${name}_link"/>
 	  </joint>
-	  <link name="${prefix_frame}_link">
+      <link name="${name}_link">
 	      <inertial>
 	        <mass value="0.001"/>
@@ -29,9 +28,9 @@
 	  </link>
 	  <gazebo>
-	    <plugin name="${prefix_frame}_controller" filename="libhector_gazebo_ros_imu.so">
+	    <plugin name="${name}_controller" filename="libhector_gazebo_ros_imu.so">
 	       <alwaysOn>true</alwaysOn>
-	       <topicName>${prefix_topic}imu/data</topicName>
-		   <serviceName>${prefix_topic}imu/service</serviceName>
-		   <bodyName>${prefix_frame}_link</bodyName>
+	       <topicName>${name}/data</topicName>
+		   <serviceName>${name}/service</serviceName>
+		   <bodyName>${name}_link</bodyName>
 	       <updateRate>50.0</updateRate>
 	       <gaussianNoise>0.005</gaussianNoise>
