Commit message: m5013 and imu converted to new standard

File: urdf/axis_m5013.urdf.xacro (robot description, xacro)
@@ -40,5 +40,5 @@
       </collision>
     </link>
-    <joint name="joint_${name}_pan" type="revolute">
+    <joint name="${name}_pan_joint" type="revolute">
       <axis xyz="0 0 -1"/>
       <origin xyz="0.04 0.0 0.0" rpy="0 0 0"/>
@@ -58,5 +58,5 @@
     <transmission name="${name}_pan_trans">
       <type>transmission_interface/SimpleTransmission</type>
-      <joint name="joint_${name}_pan">
+      <joint name="${name}_pan_joint">
         <hardwareInterface>PositionJointInterface</hardwareInterface>
       </joint>
@@ -66,5 +66,5 @@
       </actuator>
     </transmission>
-    <joint name="joint_${name}_tilt" type="revolute">
+    <joint name="${name}_tilt_joint" type="revolute">
       <axis xyz="0 -1 0"/>
       <origin xyz="0.0 0.0 0.0"/>
@@ -83,5 +83,5 @@
     <transmission name="${name}_tilt_trans">
       <type>transmission_interface/SimpleTransmission</type>
-      <joint name="joint_${name}_tilt">
+      <joint name="${name}_tilt_joint">
         <hardwareInterface>PositionJointInterface</hardwareInterface>
       </joint>

File: urdf/imu.urdf.xacro (robot description, xacro)
@@ -1,5 +1,5 @@
 <?xml version="1.0"?>
 <robot name="sensor_imu" xmlns:xacro="http://www.ros.org/wiki/xacro">
-  <xacro:macro name="sensor_imu" params="name prefix_frame prefix_topic parent *origin">
+  <xacro:macro name="sensor_imu" params="name parent *origin">
 	  <joint name="${name}_joint" type="fixed">
 	      <axis xyz="1 0 0"/>
@@ -7,5 +7,5 @@
 	      <xacro:insert_block name="origin"/>
 	      <parent link="${parent}"/>
-	      <child link="${prefix_frame}_link"/>
+	      <child link="${name}_link"/>
 	  </joint>
 	  <link name="${name}_link">
@@ -30,7 +30,7 @@
 	  <gazebo>
 	    <plugin name="${name}_controller" filename="libgazebo_ros_imu.so">
-	       <topicName>${prefix_topic}/data</topicName>
-		   <serviceName>${prefix_topic}/service</serviceName>
-		   <bodyName>${prefix_frame}_link</bodyName>
+	       <topicName>${name}/data</topicName>
+		   <serviceName>${name}/service</serviceName>
+		   <bodyName>${name}_link</bodyName>
 	       <gaussianNoise>0.005</gaussianNoise>
 	    </plugin>
