Commit message: update

File: urdf/axis_m5525.urdf.xacro (robot description, xacro)
@@ -69,5 +69,5 @@
     <joint name="${prefix}_tilt_joint" type="revolute">
       <axis xyz="0 -1 0"/>
-      <origin xyz="0.0 0.0 0.0" rpy="0 ${PI/2} 0"/>
+      <origin xyz="0.0 0.0 0.0" rpy="0 ${-PI/2} 0"/>
       <parent link="${prefix}_pan_link"/>
       <child link="${prefix}_tilt_link"/>
@@ -118,5 +118,5 @@
     </link>
     <gazebo reference="${prefix}_base_link">
-      <material>Gazebo/DarkGrey</material>
+      <material>Gazebo/FlatBlack</material>
     </gazebo>
     <!-- Axis sensor for simulation -->

File: urdf/benewake_ce30.urdf.xacro (robot description, xacro)
@@ -57,5 +57,5 @@
       <xacro:unless value="${gpu}">
         <xacro:property name="ray_type" value="ray" />
-        <xacro:property name="plugin_lib" value="libgazebo_ros_velodyne_laser.so" />
+        <xacro:property name="plugin_lib" value="libgazebo_ros_block_laser.so" />
       </xacro:unless>
         <sensor type="${ray_type}" name="${prefix}_sensor">

File: urdf/hokuyo3d.urdf.xacro (robot description, xacro)
@@ -45,5 +45,5 @@
       <xacro:unless value="${gpu}">
         <xacro:property name="ray_type" value="ray" />
-        <xacro:property name="plugin_lib" value="libgazebo_ros_velodyne_laser.so" />
+        <xacro:property name="plugin_lib" value="libgazebo_ros_block_laser.so" />
       </xacro:unless>
       <sensor type="${ray_type}" name="${prefix}_sensor">

File: urdf/hokuyo_utm30lx.urdf.xacro (robot description, xacro)
@@ -13,5 +13,5 @@
     <link name="${prefix}_base_link">
       <visual>
-        <origin xyz="0 0 0.055" rpy="0 0 0"/>
+        <origin xyz="0 0 0" rpy="0 0 0"/>
         <geometry>
             <mesh filename="package://robotnik_sensors/meshes/hokuyo_utm_30lx.dae"/>

File: urdf/imu.urdf.xacro (robot description, xacro)
@@ -1,44 +1,59 @@
 <?xml version="1.0"?>
 <robot name="sensor_imu" xmlns:xacro="http://wiki.ros.org/xacro">
-  <xacro:macro name="sensor_imu" params="prefix ns:='' parent *origin prefix_topic:='imu'">
+  <xacro:macro name="sensor_imu" params="prefix ns:='' parent *origin">
 	  <joint name="${prefix}_joint" type="fixed">
-      <axis xyz="1 0 0"/>
-      <!--origin xyz="0 0 0.2825"/-->
-      <xacro:insert_block name="origin"/>
-      <parent link="${parent}"/>
-      <child link="${prefix}_link"/>
+	      <axis xyz="1 0 0"/>
+	      <!--origin xyz="0 0 0.2825"/-->
+	      <xacro:insert_block name="origin"/>
+	      <parent link="${parent}"/>
+	      <child link="${prefix}_link"/>
 	  </joint>
-    <link name="${prefix}_link">
-      <inertial>
-        <mass value="0.001"/>
-        <origin rpy="0 0 0" xyz="0 0 0"/>
-        <inertia ixx="0.00000000167" ixy="0" ixz="0" iyy="0.00000000167" iyz="0" izz="0.00000000167"/>
-      </inertial>
-      <visual>
-        <origin rpy="0 0 0" xyz="0 0 0"/>
-        <geometry>
-          <box size="0.001 0.001 0.001"/>
-        </geometry>
-      </visual>
-    </link>
-    <gazebo reference="${prefix}_link">
-      <gravity>true</gravity>
-      <sensor name="${prefix}_imu_sensor" type="imu">
-        <always_on>true</always_on>
-        <update_rate>100</update_rate>
-        <visualize>true</visualize>
-        <topic>__default_topic__</topic>
-        <plugin filename="libgazebo_ros_imu_sensor.so" name="${prefix}_imu_plugin">
-          <topicName>${prefix_topic}/data_raw</topicName>
-  		    <bodyName>${prefix}_link</bodyName>
-          <updateRateHZ>100.0</updateRateHZ>
-          <gaussianNoise>0.0</gaussianNoise>
-          <xyzOffset>0 0 0</xyzOffset>
-          <rpyOffset>0 0 0</rpyOffset>
-  		    <frameName>${prefix}_link</frameName>
-        </plugin>
-        <pose>0 0 0 0 0 0</pose>
-      </sensor>
-    </gazebo>
+	  <link name="${prefix}_link">
+	      <inertial>
+	        <mass value="0.001"/>
+	        <origin rpy="0 0 0" xyz="0 0 0"/>
+	        <inertia ixx="0.00000000167" ixy="0" ixz="0" iyy="0.00000000167" iyz="0" izz="0.00000000167"/>
+	      </inertial>
+	      <visual>
+	        <origin rpy="0 0 0" xyz="0 0 0"/>
+	        <geometry>
+	          <box size="0.001 0.001 0.001"/>
+	        </geometry>
+	      </visual>
+	      <!--collision>
+	        <origin rpy="0 0 0" xyz="0 0 0"/>
+	        <geometry>
+	          <box size=".001 .001 .001"/>
+	        </geometry>
+	      </collision-->
+	  </link>
+	  <!--<gazebo>-->
+		<!--<plugin name="${prefix}_controller" filename="libgazebo_ros_imu.so">-->
+		   <!--<topicName>${ns}imu/data</topicName>-->
+		   <!--<serviceName>imu/service</serviceName>-->
+		   <!--<bodyName>${prefix}_link</bodyName>-->
+		   <!--<updateRateHZ>50.0</updateRateHZ>-->
+		   <!--<gaussianNoise>0.0</gaussianNoise>-->
+		<!--</plugin>-->
+	  <!--</gazebo>-->
+ <gazebo reference="${prefix}_link">
+    <gravity>true</gravity>
+    <sensor name="${prefix}_imu_sensor" type="imu">
+      <always_on>true</always_on>
+      <update_rate>100</update_rate>
+      <visualize>true</visualize>
+      <topic>__default_topic__</topic>
+      <plugin filename="libgazebo_ros_imu_sensor.so" name="${prefix}_imu_plugin">
+        <topicName>imu/data</topicName>
+		<bodyName>${prefix}_link</bodyName>
+        <updateRateHZ>100.0</updateRateHZ>
+        <gaussianNoise>0.0</gaussianNoise>
+        <xyzOffset>0 0 0</xyzOffset>
+        <rpyOffset>0 0 0</rpyOffset>
+		<frameName>${prefix}_link</frameName>
+      </plugin>
+      <pose>0 0 0 0 0 0</pose>
+    </sensor>
+  </gazebo>
   </xacro:macro>
 </robot>

File: urdf/imu_hector_plugin.urdf.xacro (robot description, xacro)
@@ -1,51 +1,51 @@
 <?xml version="1.0"?>
 <robot name="sensor_imu" xmlns:xacro="http://wiki.ros.org/xacro">
-  <xacro:macro name="sensor_imu_hector" params="prefix parent *origin prefix_topic:='imu'">
+  <xacro:macro name="sensor_imu_hector" params="prefix parent *origin">
 	  <joint name="${prefix}_joint" type="fixed">
-      <axis xyz="1 0 0"/>
-      <!--origin xyz="0 0 0.2825"/-->
-      <xacro:insert_block name="origin"/>
-      <parent link="${parent}"/>
-      <child link="${prefix}_link"/>
+	      <axis xyz="1 0 0"/>
+	      <!--origin xyz="0 0 0.2825"/-->
+	      <xacro:insert_block name="origin"/>
+	      <parent link="${parent}"/>
+	      <child link="${prefix}_link"/>
 	  </joint>
 	  <link name="${prefix}_link">
-      <inertial>
-        <mass value="0.001"/>
-        <origin rpy="0 0 0" xyz="0 0 0"/>
-        <inertia ixx="0.0001" ixy="0" ixz="0" iyy="0.000001" iyz="0" izz="0.0001"/>
-      </inertial>
-      <visual>
-        <origin rpy="0 0 0" xyz="0 0 0"/>
-        <geometry>
-          <box size="0.001 0.001 0.001"/>
-        </geometry>
-      </visual>
-      <collision>
-        <origin rpy="0 0 0" xyz="0 0 0"/>
-        <geometry>
-          <box size=".001 .001 .001"/>
-        </geometry>
-      </collision>
+	      <inertial>
+	        <mass value="0.001"/>
+	        <origin rpy="0 0 0" xyz="0 0 0"/>
+	        <inertia ixx="0.0001" ixy="0" ixz="0" iyy="0.000001" iyz="0" izz="0.0001"/>
+	      </inertial>
+	      <visual>
+	        <origin rpy="0 0 0" xyz="0 0 0"/>
+	        <geometry>
+	          <box size="0.001 0.001 0.001"/>
+	        </geometry>
+	      </visual>
+	      <collision>
+	        <origin rpy="0 0 0" xyz="0 0 0"/>
+	        <geometry>
+	          <box size=".001 .001 .001"/>
+	        </geometry>
+	      </collision>
 	  </link>
 	  <gazebo>
 	    <plugin name="${prefix}_controller" filename="libhector_gazebo_ros_imu.so">
-       <alwaysOn>true</alwaysOn>
-       <topicName>${prefix_topic}/data_raw</topicName>
-  	   <serviceName>${prefix}imu/service</serviceName>
-  	   <bodyName>${prefix}_link</bodyName>
-  	   <frameId>${prefix}_link</frameId>
-       <updateRate>50.0</updateRate>
-       <gaussianNoise>0.00</gaussianNoise>
-       <yawOffset>0.0</yawOffset>
-       <yawDrift>0.0</yawDrift>
-       <yawGaussianNoise>0.0</yawGaussianNoise>
-       <!-- angular velocities parameters -->
-       <rateOffset>0.0 0.0 0.0</rateOffset>
-       <rateDrift>0.0 0.0 0.0</rateDrift>
-       <rateGaussianNoise>0.0 0.0 0.0</rateGaussianNoise>
-       <!-- linear accelerations parameters -->
-       <accelOffset>0.0 0.0 0.0</accelOffset>
-       <accelDrift>0.0 0.0 0.0</accelDrift>
-       <accelGaussianNoise>0.0 0.0 0.0</accelGaussianNoise>
+	       <alwaysOn>true</alwaysOn>
+	       <topicName>imu/data</topicName>
+		   <serviceName>${prefix}imu/service</serviceName>
+		   <bodyName>${prefix}_link</bodyName>
+		   <frameId>${prefix}_link</frameId>
+	       <updateRate>50.0</updateRate>
+	       <gaussianNoise>0.00</gaussianNoise>
+           <yawOffset>0.0</yawOffset>
+           <yawDrift>0.0</yawDrift>
+           <yawGaussianNoise>0.0</yawGaussianNoise>
+           <!-- angular velocities parameters -->
+           <rateOffset>0.0 0.0 0.0</rateOffset>
+           <rateDrift>0.0 0.0 0.0</rateDrift>
+           <rateGaussianNoise>0.0 0.0 0.0</rateGaussianNoise>
+           <!-- linear accelerations parameters -->
+           <accelOffset>0.0 0.0 0.0</accelOffset>
+           <accelDrift>0.0 0.0 0.0</accelDrift>
+           <accelGaussianNoise>0.0 0.0 0.0</accelGaussianNoise>
 	    </plugin>
 	  </gazebo>

File: urdf/ouster1.urdf.xacro (robot description, xacro)
@@ -49,5 +49,5 @@
       <xacro:unless value="${gpu}">
         <xacro:property name="ray_type" value="ray" />
-        <xacro:property name="plugin_lib" value="libgazebo_ros_velodyne_laser.so" />
+        <xacro:property name="plugin_lib" value="libgazebo_ros_block_laser.so" />
       </xacro:unless>
       <sensor type="${ray_type}" name="${prefix}_sensor">

File: urdf/rs_bpearl.urdf.xacro (robot description, xacro)
@@ -50,5 +50,5 @@
       <xacro:unless value="${gpu}">
         <xacro:property name="ray_type" value="ray" />
-        <xacro:property name="plugin_lib" value="libgazebo_ros_velodyne_laser.so" />
+        <xacro:property name="plugin_lib" value="libgazebo_ros_block_laser.so" />
       </xacro:unless>
         <sensor type="${ray_type}" name="${prefix}_sensor">

File: urdf/rslidar.urdf.xacro (robot description, xacro)
@@ -49,5 +49,5 @@
       <xacro:unless value="${gpu}">
         <xacro:property name="ray_type" value="ray" />
-        <xacro:property name="plugin_lib" value="libgazebo_ros_velodyne_laser.so" />
+        <xacro:property name="plugin_lib" value="libgazebo_ros_block_laser.so" />
       </xacro:unless>
         <sensor type="${ray_type}" name="${prefix}_sensor">
@@ -79,5 +79,5 @@
           </ray>
           <plugin name="${prefix}_controller" filename="${plugin_lib}">
-            <topicName>${prefix_topic}/point_cloud</topicName>
+            <topicName>${prefix_topic}/points</topicName>
             <frameName>/${prefix}_link</frameName>
             <gaussianNoise>0.008</gaussianNoise>

File: urdf/rslidar_mems.urdf.xacro (robot description, xacro)
@@ -33,55 +33,4 @@
     </joint>
     <link name="${prefix}_link"/>
-    <!-- sensor for simulation -->
-    <sensor_rslidar_mems_gazebo range_min="1" range_max="180" gpu="false" />
-  </xacro:macro>
-  <xacro:macro name="sensor_rslidar_mems_gazebo" params="range_min range_max gpu">
-    <gazebo reference="${prefix}_link">
-      <xacro:if value="${gpu}">
-        <!-- Using GPU needs: https://github.com/RobotnikAutomation/velodyne_simulator -->
-        <xacro:property name="ray_type" value="gpu_ray" />
-        <xacro:property name="plugin_lib" value="libgazebo_ros_velodyne_gpu_laser.so" />
-      </xacro:if>
-      <xacro:unless value="${gpu}">
-        <xacro:property name="ray_type" value="ray" />
-        <xacro:property name="plugin_lib" value="libgazebo_ros_velodyne_laser.so" />
-      </xacro:unless>
-      <sensor type="${ray_type}" name="${prefix}_sensor">
-          <pose>0 0 0 0 0 0</pose>
-          <visualize>false</visualize>
-          <update_rate>15</update_rate>
-          <ray>
-              <scan>
-                  <horizontal>
-                      <samples>100</samples>
-                      <resolution>1.0</resolution>
-                      <min_angle>-1.0472</min_angle>
-                      <max_angle>1.0472</max_angle>
-                  </horizontal>
-                  <vertical>
-                      <samples>100</samples>
-                      <resolution>1.0</resolution>
-                      <min_angle>-0.610865238</min_angle>
-                      <max_angle>1.83591184</max_angle>
-                  </vertical>
-              </scan>
-              <range>
-              <min>${range_min}</min>
-              <max>${range_max}</max>
-                  <resolution>0.0035</resolution>
-              </range>
-              <noise>
-                  <type>gaussian</type>
-                  <mean>0.0</mean>
-                  <stddev>0.01</stddev>
-              </noise>
-          </ray>
-          <plugin name="${prefix}_controller" filename="${plugin_lib}">
-              <topicName>/robot/front_3d_laser/point_cloud</topicName>
-              <frameName>/${prefix}_link</frameName>
-              <ignoreTfPrefix>1</ignoreTfPrefix>
-          </plugin>
-      </sensor>
-    </gazebo>
   </xacro:macro>
 </robot>

File: urdf/sick_s300.urdf.xacro (robot description, xacro)
@@ -2,8 +2,9 @@
 <robot name="sensor_sick_s300" xmlns:xacro="http://wiki.ros.org/xacro">
   <xacro:macro name="sensor_sick_s300" params="prefix parent prefix_topic:='front_laser' *origin min_angle:=-2.3562 max_angle:=2.3562 gpu:=^|true">
-    <joint name="${prefix}_base_joint" type="fixed">
+    <joint name="${prefix}_base_joint" type="revolute">
       <xacro:insert_block name="origin" />
       <parent link="${parent}"/>
       <child link="${prefix}_base_link"/>
+      <limit effort="100" velocity="100" lower="0.0" upper="0.0"/>
 	</joint>
 	<link name="${prefix}_base_link">
@@ -39,4 +40,14 @@
 	</joint>
 	<link name="${prefix}_link" />
+	<transmission name="${prefix}_base_trans">
+      <type>transmission_interface/SimpleTransmission</type>
+      <joint name="${prefix}_base_joint">
+        <hardwareInterface>hardware_interface/VelocityJointInterface</hardwareInterface>
+      </joint>
+      <actuator name="sick_motor">
+        <hardwareInterface>hardware_interface/VelocityJointInterface</hardwareInterface>
+        <mechanicalReduction>${ptz_mechanical_reduction}</mechanicalReduction>
+      </actuator>
+    </transmission>
 	<!-- Sick sensor sensor for simulation -->
 	<sensor_sick_s300_gazebo />

File: urdf/ueye_cp_gige.urdf.xacro (robot description, xacro)
@@ -3,5 +3,5 @@
   <xacro:macro name="sensor_ueye_cp_gige" params="prefix parent *origin">
     <joint name="${prefix}_joint" type="fixed">
-      <xacro:insert_block name="origin"/>
+      <insert_block name="origin"/>
       <parent link="${parent}"/>
       <child link="${prefix}_base_link"/>

File: urdf/velodyne_vlp16.urdf.xacro (robot description, xacro)
@@ -45,5 +45,5 @@
       <xacro:unless value="${gpu}">
         <xacro:property name="ray_type" value="ray" />
-        <xacro:property name="plugin_lib" value="libgazebo_ros_velodyne_laser.so" />
+        <xacro:property name="plugin_lib" value="libgazebo_ros_block_laser.so" />
       </xacro:unless>
       <sensor type="${ray_type}" name="${prefix}_sensor">
